Commit message: fix(urdfs): Add proper joint limits

File: src/urdfs/airbot_play_inspire_eg2_4c_compatible_v1/urdf/airbot_play_inspire_eg2_4c_compatible_v1.urdf (robot description, URDF)
Before this commit: robot airbot_play_inspire_eg2_4c_compatible_v1, 12 links, 11 joints
Joints:
- joint joint1: limit lower=-10 upper=10 effort=100 velocity=110 -> lower=-2 upper=3.14 effort=100 velocity=110
- joint joint2: limit lower=-10 upper=10 effort=100 velocity=110 -> lower=-3.14 upper=0 effort=100 velocity=110
- joint joint3: limit lower=-10 upper=10 effort=100 velocity=110 -> lower=0 upper=3.9 effort=100 velocity=110
- joint joint4: limit lower=-10 upper=10 effort=100 velocity=110 -> lower=-1.8 upper=1.57 effort=100 velocity=110
- joint joint5: limit lower=-10 upper=10 effort=100 velocity=110 -> lower=-1.4 upper=1.57 effort=100 velocity=110
- joint joint6: limit lower=-10 upper=10 effort=100 velocity=1000 -> lower=-1.57 upper=1.57 effort=100 velocity=1000
