Commit message: feat(*):add airbot play v1 config

File: src/moveit_configs/airbot_play_v1_config/config/gazebo_airbot_play_v1.urdf (robot description, URDF)
Before this commit: robot ARX-5s-V5.0-urdf ceshi3, 7 links, 6 joints
Links:
- removed link link6
- added link custom_end_link, mass 1E-15
- added link gripper_link, mass 1E-15
- link link1: mass 0.051342 -> 0.078163
- link link2: mass 1.1379 -> 1.0604
- link link3: mass 0.55615 -> 0.55999
- link link4: mass 0.35037 -> 0.34333
- link link5: mass 0.33138 -> 0.33126
Joints:
- added joint joint_custom_end: type fixed, parent gripper_link, child custom_end_link, origin xyz=0 0 0.078 rpy=1.5708 -1.5708 0
- joint joint1: limit lower=-10 upper=10 effort=100 velocity=1000 -> lower=-10 upper=10 effort=100 velocity=110; origin xyz=0 0 0 rpy=0 0 0 -> xyz=0 0 0.1005 rpy=0 0 0
- joint joint2: limit lower=-10 upper=10 effort=100 velocity=1000 -> lower=-10 upper=10 effort=100 velocity=110; origin xyz=0 0 0.0402 rpy=-1.5708 0.0016463 3.1416 -> xyz=0 0 0 rpy=-1.5708 0 3.1416
- joint joint3: limit lower=-10 upper=10 effort=100 velocity=1000 -> lower=-10 upper=10 effort=100 velocity=110; origin xyz=0.264 0 0 rpy=0 0 -2.9169 -> xyz=0.264 0 0 rpy=0 0 -2.9159
- joint joint4: limit lower=-10 upper=10 effort=100 velocity=1000 -> lower=-10 upper=10 effort=100 velocity=110; origin xyz=0.25132 0 0 rpy=0 0 -0.22636 -> xyz=0.25137 0 -0.002 rpy=0 0 -0.22569
- joint joint5: limit lower=-10 upper=10 effort=100 velocity=1000 -> lower=-10 upper=10 effort=100 velocity=110; origin xyz=0.06 -0.0005 -0.002 rpy=-1.5708 -0.0025284 0 -> xyz=0.06 0 0 rpy=-1.5708 -1.5708 0
- joint joint6: axis 1 0 0 -> 0 0 1; child link6 -> gripper_link; origin xyz=0.075 0 0 rpy=0 0 0 -> xyz=0 0 0 rpy=-1.5708 0 0
